Commit message: Move model via commands

File: src/ags_description/urdf/ags.xacro (robot description, xacro)
@@ -269,3 +269,51 @@
         </inertial>
     </link>
+    <!-- ================= ROS2 CONTROL ================= -->
+    <ros2_control name="nexus_ags_controller" type="system">
+        <hardware>
+            <plugin>gz_ros2_control/GazeboSimSystem</plugin>
+        </hardware>
+        <joint name="shoulder_joint">
+            <command_interface name="position" />
+            <state_interface name="position" />
+            <state_interface name="velocity" />
+        </joint>
+        <joint name="elbow_joint">
+            <command_interface name="position" />
+            <state_interface name="position" />
+            <state_interface name="velocity" />
+        </joint>
+        <joint name="forearm_joint">
+            <command_interface name="position" />
+            <state_interface name="position" />
+            <state_interface name="velocity" />
+        </joint>
+        <joint name="wrist_pitch_joint">
+            <command_interface name="position" />
+            <state_interface name="position" />
+            <state_interface name="velocity" />
+        </joint>
+        <joint name="wrist_roll_joint">
+            <command_interface name="position" />
+            <state_interface name="position" />
+            <state_interface name="velocity" />
+        </joint>
+        <joint name="left_finger_joint">
+            <command_interface name="position" />
+            <state_interface name="position" />
+            <state_interface name="velocity" />
+        </joint>
+        <joint name="right_finger_joint">
+            <command_interface name="position" />
+            <state_interface name="position" />
+            <state_interface name="velocity" />
+        </joint>
+    </ros2_control>
+    <!-- ================= GAZEBO ================= -->
+    <gazebo>
+        <plugin filename="libgz_ros2_control-system.so"
+            name="gz_ros2_control::GazeboSimROS2ControlPlugin">
+            <parameters>/home/madhu/ros2_nexus_ags_ws/install/ags_description/share/ags_description/config/controllers.yaml</parameters>
+        </plugin>
+    </gazebo>
 </robot>

Commit message: Add camera and see the object

File: src/ags_description/urdf/ags.xacro (robot description, xacro)
@@ -209,4 +209,20 @@
         </inertial>
     </link>
+    <!-- GRIPPER BASE to CAMERA -->
+    <joint name="camera_joint" type="fixed">
+        <parent link="gripper_base" />
+        <child link="camera_link" />
+        <origin xyz="0 0 0.08" rpy="0 -1.57 0" />
+    </joint>
+    <link name="camera_link">
+        <visual>
+            <geometry>
+                <box size="0.04 0.04 0.04" />
+            </geometry>
+            <material name="black">
+                <color rgba="0 0 0 1" />
+            </material>
+        </visual>
+    </link>
     <!-- GRIPPER BASE to LEFT FINGER -->
     <joint name="left_finger_joint" type="prismatic">
@@ -269,4 +285,26 @@
         </inertial>
     </link>
+    <!-- CAMERA PLUGIN -->
+    <gazebo reference="camera_link">
+        <sensor name="camera" type="camera">
+            <update_rate>30</update_rate>
+            <topic>camera/image</topic>
+            <camera>
+                <horizontal_fov>1.396</horizontal_fov>
+                <image>
+                    <width>640</width>
+                    <height>480</height>
+                    <format>R8G8B8</format>
+                </image>
+            </camera>
+        </sensor>
+    </gazebo>
+    <gazebo>
+        <plugin
+            filename="gz-sim-sensors-system"
+            name="gz::sim::systems::Sensors">
+            <render_engine>ogre2</render_engine>
+        </plugin>
+    </gazebo>
     <!-- ================= ROS2 CONTROL ================= -->
     <ros2_control name="nexus_ags_controller" type="system">
@@ -314,5 +352,6 @@
         <plugin filename="libgz_ros2_control-system.so"
             name="gz_ros2_control::GazeboSimROS2ControlPlugin">
-            <parameters>/home/madhu/ros2_nexus_ags_ws/install/ags_description/share/ags_description/config/controllers.yaml</parameters>
+            <parameters>
+                /home/madhu/ros2_nexus_ags_ws/install/ags_description/share/ags_description/config/controllers.yaml</parameters>
         </plugin>
     </gazebo>

Commit message: elbow rotation fix

File: src/ags_description/urdf/ags.xacro (robot description, xacro)
@@ -67,5 +67,5 @@
         <origin xyz="0 0 0.4" />
         <axis xyz="1 0 0" />
-        <limit lower="0" upper="3.14" effort="300" velocity="1" />
+        <limit lower="-1.57" upper="1.57" effort="300" velocity="1" />
     </joint>
     <link name="elbow_link">
